File: clock_logic.kicad_sch (KiCad schematic)
At the start: 7 parts, among them SW1 SW_Push_SPDT

Commit message: Fix non standard switch buton
Connections:
- net GND: now also SW1.6 (B); no longer SW1.2 (B)
- net at R3.2, U2.2 (TRIG): now also SW1.5 (A); no longer SW1.1 (A)
- net at R6.2, U2.4 (RESET): now also SW1.4 (C); no longer SW1.3 (C)
Changed lines of the file:
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@@
       (effects (font (size 1.27 1.27)) hide)
     )
-    (pin "1")
-    (pin "3")
-    (pin "2")
+    (pin "6")
+    (pin "4")
+    (pin "5")
     (instances
       (project "clock"
